File: pcb/main_v2/oscillator.kicad_sch (KiCad schematic)
At the start: 25 parts, among them IC501 SPF5043Z, IC502 PD0922J5050S2HF, IC503 SPF5043Z, U501 XMB0220K1-50100G, Y501 ASGTX-P-1.500GHZ-1

Commit message: updated schematic after review
Connections:
- net Carrier Frequency: Rx renamed Oscillator Rx
- net Carrier Frequency: Tx renamed Oscillator Tx
Other:
- note added: "f_c = 1.5 GHz"
Changed lines of the file:
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@@
+		)
+	)
+	(text "f_c = 1.5 GHz"
+		(exclude_from_sim no)
+		(at 210.82 113.03 0)
+		(effects
+			(font
+				(size 1.27 1.27)
+			)
 		)
 	)
@@
 		(exclude_from_sim no)
 		(at 101.346 42.418 0)
+		(effects
+			(font
+				(size 1.27 1.27)
+			)
+		)
+	)
+	(text "f_c = 1.5 GHz"
+		(exclude_from_sim no)
+		(at 216.408 150.876 0)
 		(effects
 			(font
@@
 	(wire
 		(pts
-			(xy 198.12 115.57) (xy 195.58 115.57)
+			(xy 205.74 115.57) (xy 195.58 115.57)
 		)
 		(stroke
@@
 		)
 	)
+	(label "f_c = 1.5 GHz"
+		(at 60.96 63.5 270)
+		(effects
+			(font
+				(size 1.27 1.27)
+			)
+			(justify right bottom)
+		)
+	)
 	(label "filtered XO 1"
 		(at 99.06 123.19 180)
@@
 		)
 	)
-	(global_label "Carrier Frequency: Tx"
+	(hierarchical_label "Oscillator Rx"
 		(shape input)
-		(at 204.47 153.67 0)
+		(at 198.12 115.57 90)
 		(fields_autoplaced yes)
 		(effects
@@
 			(justify left)
 		)
-		(property "Intersheetrefs" "${INTERSHEET_REFS}"
-			(at 228.0171 153.67 0)
-			(hide yes)
-			(show_name no)
-			(do_not_autoplace no)
-			(effects
-				(font
-					(size 1.27 1.27)
+		(property "Netzklasse" "High Speed 50Ohm"
+			(at 199.39 115.57 90)
+			(show_name no)
+			(do_not_autoplace no)
+			(effects
+				(font
+					(size 1.27 1.27)
+					(italic yes)
 				)
 				(justify left)
 			)
 		)
-		(property "Net Class" "High Speed 50Ohm"
-			(at 204.47 157.5118 0)
-			(hide yes)
-			(show_name no)
-			(do_not_autoplace no)
-			(effects
-				(font
-					(size 1.27 1.27)
+	)
+	(hierarchical_label "Oscillator Tx"
+		(shape input)
+		(at 200.66 153.67 90)
+		(fields_autoplaced yes)
+		(effects
+			(font
+				(size 1.27 1.27)
+			)
+			(justify left)
+		)
+		(property "Netzklasse" "High Speed 50Ohm"
+			(at 201.93 153.67 90)
+			(show_name no)
+			(do_not_autoplace no)
+			(effects
+				(font
+					(size 1.27 1.27)
+					(italic yes)
 				)
 				(justify left)
-			)
-		)
-	)
-	(global_label "Carrier Frequency: Rx"
-		(shape input)
-		(at 198.12 115.57 0)
-		(fields_autoplaced yes)
-		(effects
-			(font
-				(size 1.27 1.27)
-			)
-			(justify left)
-		)
-		(property "Intersheetrefs" "${INTERSHEET_REFS}"
-			(at 221.9695 115.57 0)
-			(hide yes)
-			(show_name no)
-			(do_not_autoplace no)
-			(effects
-				(font
-					(size 1.27 1.27)
-				)
-				(justify left)
-			)
-		)
-		(property "Net Class" "High Speed 50Ohm"
-			(at 198.12 119.4118 0)
-			(hide yes)
-			(show_name no)
-			(do_not_autoplace no)
-			(effects
-				(font
-					(size 1.27 1.27)
-				)
-				(justify left)

Commit message: added new osci
Changed lines of the file:
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@@
 	(text "Low Pass"
 		(exclude_from_sim no)
-		(at 240.538 78.486 0)
+		(at 213.106 70.104 0)
 		(effects
 			(font
@@
 	(text "f_c = 1.5 GHz"
 		(exclude_from_sim no)
-		(at 210.82 113.03 0)
+		(at 206.756 110.744 0)
 		(effects
 			(font
@@
 	(wire
 		(pts
+			(xy 209.55 115.57) (xy 195.58 115.57)
+		)
+		(stroke
+			(width 0)
+			(type default)
+		)
+	)
+	(wire
+		(pts
 			(xy 152.4 54.61) (xy 138.43 54.61)
 		)
@@
 	(wire
 		(pts
+			(xy 209.55 114.3) (xy 209.55 115.57)
+		)
+		(stroke
+			(width 0)
+			(type default)
+		)
+	)
+	(wire
+		(pts
 			(xy 78.74 135.89) (xy 92.71 135.89)
 		)
@@
 	(wire
 		(pts
+			(xy 212.09 114.3) (xy 209.55 114.3)
+		)
+		(stroke
+			(width 0)
+			(type default)
+		)
+	)
+	(wire
+		(pts
 			(xy 120.65 132.08) (xy 132.08 132.08)
 		)
@@
 	(wire
 		(pts
-			(xy 205.74 115.57) (xy 195.58 115.57)
-		)
-		(stroke
-			(width 0)
-			(type default)
-		)
-	)
-	(wire
-		(pts
 			(xy 78.74 140.97) (xy 99.06 140.97)
 		)
@@
 	(wire
 		(pts
+			(xy 210.82 45.72) (xy 222.25 45.72)
+		)
+		(stroke
+			(width 0)
+			(type default)
+		)
+	)
+	(wire
+		(pts
+			(xy 99.06 118.11) (xy 110.49 118.11)
+		)
+		(stroke
+			(width 0)
+			(type default)
+		)
+	)
+	(wire
+		(pts
+			(xy 34.29 138.43) (xy 43.18 138.43)
+		)
+		(stroke
+			(width 0)
+			(type default)
+		)
+	)
+	(wire
+		(pts
 			(xy 204.47 153.67) (xy 199.39 153.67)
-		)
-		(stroke
-			(width 0)
-			(type default)
-		)
-	)
-	(wire
-		(pts
-			(xy 210.82 45.72) (xy 222.25 45.72)
-		)
-		(stroke
-			(width 0)
-			(type default)
-		)
-	)
-	(wire
-		(pts
-			(xy 99.06 118.11) (xy 110.49 118.11)
-		)
-		(stroke
-			(width 0)
-			(type default)
-		)
-	)
-	(wire
-		(pts
-			(xy 34.29 138.43) (xy 43.18 138.43)
 		)
 		(stroke
@@
 	(hierarchical_label "Oscillator Rx"
 		(shape input)
-		(at 198.12 115.57 90)
-		(fields_autoplaced yes)
+		(at 212.09 114.3 0)
 		(effects
 			(font
@@
 			(justify left)
 		)
-		(property "Netzklasse" "High Speed 50Ohm"
-			(at 199.39 115.57 90)
-			(show_name no)
-			(do_not_autoplace no)
-			(effects
-				(font
-					(size 1.27 1.27)
-					(italic yes)
-				)
-				(justify left)
+		(property "Net Class" "High Speed 50Ohm"
+			(at 217.17 117.348 0)
+			(show_name no)
+			(do_not_autoplace no)
+			(effects
+				(font
+					(size 1.27 1.27)
+					(italic yes)
+				)
 			)
 		)
@@
 	(hierarchical_label "Oscillator Tx"
 		(shape input)
-		(at 200.66 153.67 90)
-		(fields_autoplaced yes)
+		(at 204.47 153.67 0)
 		(effects
 			(font
@@
 			(justify left)
 		)
-		(property "Netzklasse" "High Speed 50Ohm"
-			(at 201.93 153.67 90)
-			(show_name no)
-			(do_not_autoplace no)
-			(effects
-				(font
-					(size 1.27 1.27)
-					(italic yes)
-				)
-				(justify left)
-			)
-		)
+		(property "Net Class" "High Speed 50Ohm"
+			(at 214.122 155.702 0)
+			(show_name no)
+			(do_not_autoplace no)
+			(effects
+				(font
+					(size 1.27 1.27)
+					(italic yes)
+				)
+			)
+		)

Commit message: updarted schematic and simulation
Parts:
- removed C504: 100 pF, Capacitor_SMD:C_0402_1005Metric, symbol Device:C
- removed C505, C509: 0.1 uF, Capacitor_SMD:C_0603_1608Metric, symbol Device:C
- removed C506, C507, C508, C510, C511, C512: 100 pF, Capacitor_SMD:C_0603_1608Metric, symbol Device:C
- removed FL501: LFCN-1700D+, My Footprints:LFCN1700D, symbol My Symbols:LFCN-1700D+
- removed IC501, IC503: SPF5043Z, My Footprints:SPF5043Z, symbol My Symbols:SPF5043Z
- removed IC502: PD0922J5050S2HF, My Footprints:PD0922J5050S2HF, symbol My Symbols:PD0922J5050S2HF
- removed L501, L502: 27 nH, Inductor_SMD:L_0603_1608Metric, symbol Device:L
- removed R501: 10, Resistor_SMD:R_0402_1005Metric, symbol Device:R
- removed R502, R503: 150 R, Resistor_SMD:R_0603_1608Metric, symbol Device:R
- removed R504, R505: DNI, Resistor_SMD:R_0603_1608Metric, symbol Device:R
- removed U501: XMB0220K1-50100G, My Footprints:XMB0220K1-50100G_TTT, symbol My Symbols:XMB0220K1-50100G
- removed Y501: ASGTX-P-1.500GHZ-1, My Footprints:ASGTX, symbol Libray Loder:ASGTX-P-1.500GHZ-1
- added C601, C603, C609, C610, C616, C618, C621, C623, C626: 0.1 uF, Capacitor_SMD:C_0402_1005Metric, symbol Device:C
- added C602, C604, C608, C615, C617, C619, C620, C622, C628: 10 pF, Capacitor_SMD:C_0402_1005Metric, symbol Device:C
- added C605: 2.7 nF, Capacitor_SMD:C_0402_1005Metric, symbol Device:C
- added C606: 1.2 nF, Capacitor_SMD:C_0402_1005Metric, symbol Device:C
- added C607: 39 nF, Capacitor_SMD:C_0402_1005Metric, symbol Device:C
- added C611, C612: 120 pF, Capacitor_SMD:C_0402_1005Metric, symbol Device:C
- added C613, C614: 1 nF, Capacitor_SMD:C_0402_1005Metric, symbol Device:C
- added C624, C625: 1 pF, Capacitor_SMD:C_0402_1005Metric, symbol Device:C
- added C627: DC Cut Cap, Capacitor_SMD:C_0402_1005Metric, symbol Device:C
- added D601: LED, LED_SMD:LED_0805_2012Metric, symbol Device:LED
- added L601, L602: 7.5 nH, Inductor_SMD:L_0402_1005Metric, symbol Device:L
- added R601: 51, Resistor_SMD:R_0603_1608Metric, symbol Device:R
- added R602: 4.7 k, Resistor_SMD:R_0603_1608Metric, symbol Device:R
- added R603: 360, Resistor_SMD:R_0603_1608Metric, symbol Device:R
- added R604: 680, Resistor_SMD:R_0603_1608Metric, symbol Device:R
- added R605, R606, R608, R609, R610: 10k, Resistor_SMD:R_0603_1608Metric, symbol Device:R
- added R607, R611: DNI, Resistor_SMD:R_0603_1608Metric, symbol Device:R
- added R612, R614, R615: 0, Resistor_SMD:R_0603_1608Metric, symbol Device:R
- added R613: 100, Resistor_SMD:R_0603_1608Metric, symbol Device:R
- added U601: ADF4351, Package_CSP:LFCSP-32-1EP_5x5mm_P0.5mm_EP3.25x3.25mm, symbol Timer_PLL:ADF4351
- added Y601: ATX-11-F-26.000MHZ-F05-T, My Footprints:ATX11F26000MHZF05T, symbol My Symbols:ATX-11-F-26.000MHZ-F05-T
- C501: value 100 pF -> 0.1 uF; Material C0G -> X7R; Package 0402 -> 0402; Tolerance (none) -> ±10%; Voltage (none) -> 50V
- C502: value 100 pF -> 10 pF; Material C0G -> NP0; Package 0402 -> 0402; Tolerance (none) -> ±10%; Voltage (none) -> 50V
- C503: value 100 pF -> 120 pF; Material C0G -> NP0; Package 0402 -> 0402; Tolerance (none) -> ±10%; Voltage (none) -> 50V
Connections:
- net TCX P is gone; now on net +3.3V: C503.2
- net TXC 0DC P is gone; now on net GND: C503.1
- net unbalanced OX 1 is gone; now on net GND: C501.2
- net unbalanced OX DC0 is gone; now on net +3.3V: C501.1
- net +3.3V: now also C502.1, C601.1, C602.1, C603.1, C604.1, C611.1, C612.2, C618.1, C619.1, C620.1, C621.1, C622.1, C623.1, C626.1, L601.1, L602.1, R606.2, R607.2, R612.2, U601.10 (AVDD), U601.16 (VVCO), U601.17 (VVCO), U601.28 (DVDD), U601.32 (SDVDD), U601.6 (Vp), Y601.4 (VDD)
- net GND: now also C601.2, C602.2, C603.2, C604.2, C605.1, C606.1, C608.2, C609.2, C610.2, C611.2, C612.1, C615.2, C616.2, C617.2, C618.2, C619.2, C620.2, C621.2, C622.2, C623.2, C626.2, C628.1, D601.1 (K), R601.1, R602.1, R603.1, R605.1, R608.2, R609.2, R610.2, R611.2, U601.11 (AGNDVCO), U601.18 (AGNDVCO), U601.21 (AGNDVCO), U601.27 (DGND), U601.31 (SDGND), U601.33 (EP), U601.8 (CPGND), U601.9 (AGND), Y601.1 (GND_1), Y601.2 (GND_2)
- new net: R602.2, U601.22 (RSET)
- new net: C625.1, R615.1
- new net: C616.1, C617.1, U601.19 (TEMP)
- new net: C627.2, Y601.3 (OUTPUT)
- new net: C606.2, R604.1, U601.20 (VTUNE)
- new net: C605.2, C607.2, R604.2, U601.7 (CPout)
- new net: C607.1, R603.2
- new net: C614.1, U601.29 (REFIN)
- new net: C613.1, C614.2, R601.2
- new net: R614.2, U601.12 (RF_OUT_A+)
- new net: R615.2, U601.13 (RF_OUT_A-)
- new net: C610.1, C615.1, U601.23 (VCOM)
- new net: C608.1, C609.1, U601.24 (VREF)
- new net: C624.1, R614.1
- new net: D601.2 (A), R613.2
- new net Oscillator +: C624.2, L601.2
- new net Oscillator -: C625.2, L602.2
- new net PLL: Chip Enable: R606.1, U601.4 (CE)
- new net PLL: Lock Detect: R613.1, U601.25 (LD)
- new net PLL: MUXOUT: U601.30 (MUXOUT)
- new net PLL: Power Down: R611.1, R612.1, U601.26 (PDB_RF)
- new net SPI: CLK: R608.1, U601.1 (CLK)
- new net SPI: DATA: R609.1, U601.2 (DATA)
- new net SPI: Load Enable: R607.1, R610.1, U601.3 (LE)
- new net TCXO: C613.2, C627.1, C628.2, R605.2
- no-connect marks 2 -> 3
Other:
- note added: "Eval Board: https://www.analog.com/media/en/technical-documentation/user-guides/UG-435.pdf"
- note added: "Phase Locked Loop"
- note removed: "Amplifier"
- note removed: "Balun 1:2"
- note removed: "Low Pass"
- note removed: "Output: LVPECL"
- note removed: "Power Splitter"
- note removed: "f_c = 1.5 GHz"
