File: pcb/main_v2/main_v2.kicad_pcb (KiCad board)
At the start: 4 copper layers, 179.2 x 68.5 mm, 173 parts, among them IC201 AP22811AW5-7, IC301 SE2576L-R, IC302 RMS-30+, IC401 HMC374, IC402 RMS-30+, IC601 PSA4-5043+, IC602 PSA4-5043+, IC701 74LVC244AD-Q100J, IC702 LTC6992CS6-4#TRMPBF, J101 Conn_Coaxial, J102 Conn_Coaxial, J103 Conn_Coaxial, J104 Conn_Coaxial, J105 Barrel_Jack, J701 Conn_01x03_Pin, J702 Conn_01x01_Pin, J703 Conn_01x03_Pin, J704 Conn_01x03_Pin, J705 Conn_01x01_Pin, J706 Conn_01x01_Pin, J707 Conn_01x01_Pin, J709 Conn_01x03_Pin, J710 Conn_01x03_Pin, Q201 DMP3068L-7, SW201 SW_DIP_x01, U201 LT3042xMSE, U501 ADF4351, U601 PD0922J5050D2HF, U602 XMB0220K1-50100G, U703 TXB0104D, Y501 ATX-11-F-26.000MHZ-F05-T

Commit message: update bom
Parts:
- removed FB202: 28C0236-0JW-10, Ferrite_THT:LairdTech_28C0236-0JW-10
- removed J105: Barrel_Jack, Connector_BarrelJack:BarrelJack_CUI_PJ-063AH_Horizontal_CircularHoles
- removed J710: Conn_01x03_Pin, Connector_PinHeader_2.54mm:PinHeader_1x03_P2.54mm_Vertical
- removed U703: TXB0104D, Package_SO:SOIC-14_3.9x8.7mm_P1.27mm
- added FB501: BLM18PG121SN1D, My Footprints:BLM18SP221SN1B, F.Cu at (122.8, 103.2)
- added FB502: BLM18PG121SN1D, My Footprints:BLM18SP221SN1B, F.Cu at (122.8, 105.8)
- added IC703: LTC6992CS6-4#TRMPBF, My Footprints:SOT95P280X100-6N, F.Cu at (128.0, 88.0)
- added J201: Barrel_Jack, Connector_BarrelJack:BarrelJack_CUI_PJ-063AH_Horizontal_CircularHoles, F.Cu at (30.8, 99.5)
- added J708: Conn_01x03_Pin, Connector_PinHeader_2.54mm:PinHeader_1x03_P2.54mm_Vertical, F.Cu at (123.1, 88.0)
- added R206: 10k, Resistor_SMD:R_0603_1608Metric, F.Cu at (106.3, 103.1)
- added R305: 26.7K, Resistor_SMD:R_0603_1608Metric, F.Cu at (122.8, 98.7)
- C203: value 0.1 uF -> 470u
- C204: value 120 uF -> 0.1 uF; footprint Capacitor_Tantalum_SMD:CP_EIA-6032-20_AVX-F -> Capacitor_SMD:C_0603_1608Metric
- C205: value 4.7 uF -> 120 uF; footprint Capacitor_SMD:C_0603_1608Metric -> Capacitor_Tantalum_SMD:CP_EIA-6032-20_AVX-F
- C208: value 470u -> 4.7 uF
- C301: value 1 uF -> 10 pF
- C302: value 10 pF -> 100 pF
- C303: value 1 nF -> 100 pF
- C304: value 2.2 pF -> 1 uF
- C305: value 4.7 uF -> 10 pF
- C306: value 15 pF -> 1 nF
- C307: value 100 nF -> 2.2 pF
- C308: value 3.3 pF -> 4.7 uF
- C309: value 2.4 pF -> 15 pF
- C310: value 2.4 pF -> 100 nF
- C311: value 10 pF -> 3.3 pF
- C312, C313: value 100 pF -> 2.4 pF
- C501, C504: value 0.1 uF -> 10 pF
- C502, C507, C526: value 10 pF -> 0.1 uF
- C510: value 120 pF -> 10 pF
- C511: value 10 pF -> 1 pF
- C512: value 0.1 uF -> 1 pF
- C513: value 120 pF -> 1 nF
- C514: value 1 pF -> 1 nF
- C515: value 1 pF -> 10 pF
- C516: value 1 nF -> 2.7 nF
- C517: value 1 nF -> 39 nF
- C518: value 0.1 uF -> 1.2 nF
- C520: value 2.7 nF -> 0.1 uF
- C521: value 39 nF -> 10 pF
- C522: value 1.2 nF -> 0.1 uF
- C524: value 10 pF -> 120 pF
- C525: value 0.1 uF -> 120 pF
- IC301: value SE2576L-R -> RMS-30+; footprint My Footprints:QFN50P300X300X90-17N-D -> My Footprints:RMS30
- IC302: value RMS-30+ -> SE2576L-R; footprint My Footprints:RMS30 -> My Footprints:QFN50P300X300X90-17N-D
- IC701: value 74LVC244AD-Q100J -> 74LVC4T3144PWJ; footprint My Footprints:SOIC127P1032X265-20N -> My Footprints:SOP65P640X110-14N
- IC702: value LTC6992CS6-4#TRMPBF -> 74LVC244AD-Q100J; footprint My Footprints:SOT95P280X100-6N -> My Footprints:SOIC127P1032X265-20N
- J701: value Conn_01x03_Pin -> Conn_01x05_Pin; footprint Connector_PinHeader_2.54mm:PinHeader_1x03_P2.54mm_Vertical -> Connector_PinHeader_2.54mm:PinHeader_1x05_P2.54mm_Vertical
- J702, J706: value Conn_01x01_Pin -> Conn_01x03_Pin; footprint Connector_PinHeader_2.54mm:PinHeader_1x01_P2.54mm_Vertical -> Connector_PinHeader_2.54mm:PinHeader_1x03_P2.54mm_Vertical
- J703, J709: value Conn_01x03_Pin -> Conn_01x01_Pin; footprint Connector_PinHeader_2.54mm:PinHeader_1x03_P2.54mm_Vertical -> Connector_PinHeader_2.54mm:PinHeader_1x01_P2.54mm_Vertical
- R201, R202, R303: value 1k -> 100k
- R203: value 10k -> 1k
- R205: value 453 k -> 1k
- R207: value 499 -> 453 k
- R208: value 49.9 k -> 499
- R209: value 150 -> 49.9 k
- R210: value 33.2k -> 150
- R211: value 100k -> 33.2k
- R304: value 26.7K -> 1k
- R501: value 100 -> 0
- R502, R504: value 10k -> DNI
- R505: value DNI -> 10k
- R507: value 0 -> 10k
- R508: value 0 -> 100
- R509: value DNI -> 0
- R708: value 50k -> 100R
- R712: value 100R -> 50k
- moved C601 190.0 mm to (266.2, 105.5)
- moved C603 190.0 mm to (262.2, 105.5)
- moved C605 190.0 mm to (258.3, 105.5)
- moved R601 190.0 mm to (265.9, 94.0)
- moved C408 190.0 mm to (241.5, 93.4)
- moved C501 190.0 mm to (233.5, 120.3)
- moved C502 190.0 mm to (233.5, 122.2)
- moved C503 190.0 mm to (233.5, 124.2)
- moved FL601 190.0 mm to (238.5, 114.4)
- moved IC601 190.0 mm to (237.8, 108.6)
- moved IC602 190.0 mm to (243.2, 108.6)
- moved L601 190.0 mm to (252.4, 110.6)
- moved U602 190.0 mm to (247.0, 101.2)
- moved C602 190.0 mm to (264.2, 105.5)
- moved C604 190.0 mm to (260.2, 105.5)
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Connections:
- net /power/DC Power renamed Net-(D201-K)
- C203 pad 1: +5V -> /power/USB Power
- C205 pad 1: GND -> +5V
- C205 pad 2: +3.3V -> GND
- C206 pad 1: +5V -> GND
- C206 pad 2: GND -> +3.3V
- C207 pad 1: Net-(U201-SET) -> +5V
- C208 pad 1: /power/USB Power -> Net-(U201-SET)
- C301 pad 1: GND -> Net-(IC301-LO)
- C301 pad 2: Net-(IC301-VCC1) -> /Oscillator Splitter/Oscillator Tx
- C302 pad 1: +5V -> /transmitter/Tx In
- C302 pad 2: GND -> Net-(IC301-IF)
- C303 pad 1: GND -> Net-(IC301-RF)
- C303 pad 2: +5V -> Net-(FL301-IN/OUT)
- C304 pad 1: +5V -> GND
- C304 pad 2: GND -> Net-(IC302-VCC1)
- C306 pad 1: Net-(IC301-RFOUT) -> GND
- C306 pad 2: Net-(C306-Pad2) -> +5V
- C308 pad 1: Net-(IC301-RFOUT) -> +5V
- C309 pad 1: Net-(IC301-RFOUT) -> Net-(IC302-RFOUT)
- C309 pad 2: GND -> Net-(C309-Pad2)
- C310 pad 1: /transmitter/Tx Out -> +5V
- C311 pad 1: Net-(IC302-LO) -> Net-(IC302-RFOUT)
- C311 pad 2: /Oscillator Splitter/Oscillator Tx -> GND
- C312 pad 1: /transmitter/Tx In -> Net-(IC302-RFOUT)
- C312 pad 2: Net-(IC302-IF) -> GND
- C313 pad 1: Net-(IC302-RF) -> /transmitter/Tx Out
- C313 pad 2: Net-(FL301-IN/OUT) -> GND
- C503 pad 1: +3.3V -> Net-(C503-Pad1)
- C504 pad 1: +3.3V -> Net-(C503-Pad1)
- C510 pad 1: GND -> +3.3V
- C510 pad 2: +3.3V -> GND
- C511 pad 1: +3.3V -> Net-(C511-Pad1)
- C511 pad 2: GND -> /Oscillator Splitter/Oscillator In +
- C512 pad 1: +3.3V -> Net-(C512-Pad1)
- C512 pad 2: GND -> /Oscillator Splitter/Oscillator In -
- C513 pad 1: +3.3V -> Net-(C513-Pad1)
- C513 pad 2: GND -> /Phase locked loop/TCXO
- C514 pad 1: Net-(C514-Pad1) -> Net-(U501-REFIN)
- C514 pad 2: /Oscillator Splitter/Oscillator In + -> Net-(C513-Pad1)
- C515 pad 1: Net-(C515-Pad1) -> Net-(U501-TEMP)
- C515 pad 2: /Oscillator Splitter/Oscillator In - -> GND
- C516 pad 1: Net-(C516-Pad1) -> GND
- C516 pad 2: /Phase locked loop/TCXO -> Net-(U501-CPout)
- C517 pad 1: Net-(U501-REFIN) -> Net-(C517-Pad1)
- C517 pad 2: Net-(C516-Pad1) -> Net-(U501-CPout)
- C518 pad 1: Net-(U501-TEMP) -> GND
- C518 pad 2: GND -> Net-(U501-VTUNE)
- C519 pad 1: Net-(U501-TEMP) -> Net-(U501-VCOM)
- C520 pad 1: GND -> Net-(U501-TEMP)
- C520 pad 2: Net-(U501-CPout) -> GND
- C521 pad 1: Net-(C521-Pad1) -> Net-(U501-VREF)
- C521 pad 2: Net-(U501-CPout) -> GND
- C522 pad 1: GND -> Net-(U501-VCOM)
- C522 pad 2: Net-(U501-VTUNE) -> GND
- C523 pad 1: Net-(U501-VCOM) -> Net-(U501-VREF)
- C524 pad 1: Net-(U501-VCOM) -> +3.3V
- C525 pad 1: Net-(U501-VREF) -> GND
- C525 pad 2: GND -> +3.3V
- C526 pad 1: Net-(U501-VREF) -> +3.3V
- C528 pad 2: +3.3V -> Net-(Y501-VDD)
- C529 pad 1: +3.3V -> Net-(Y501-VDD)
- C530 pad 1: +3.3V -> Net-(Y501-VDD)
- C701 pad 1: +3.3V -> Net-(IC701-VCC(A))
- D203 pad 2: Net-(D203-A) -> /power/USB Power
- D204 pad 2: /power/USB Power -> Net-(D204-A)
- FL402 pad 1: unconnected-(FL402-GROUND_1-Pad1) -> GND
- IC201 pad 3: /power/Power Faulty -> /IO Interface/Power Faulty Out
- IC201 pad 4: Net-(D203-A) -> Net-(D204-A)
- IC301 pad 1: /transmitter/Filtered Tx -> Net-(IC301-LO)
- IC301 pad 2: /IO Interface/PA Enable -> GND
- IC301 pad 4: +5V -> Net-(IC301-RF)
- IC301 pad 5: GND -> Net-(IC301-IF)
- IC302 pad 1: Net-(IC302-LO) -> /transmitter/Filtered Tx
- IC302 pad 2: GND -> /IO Interface/PA Enable
- IC302 pad 4: Net-(IC302-RF) -> +5V
- IC302 pad 5: Net-(IC302-IF) -> GND
- IC701 pad 1: GND -> Net-(IC701-VCC(A))
- IC701 pad 10: GND -> Net-(IC701-YB3)
- IC701 pad 11: Net-(IC701-2A3) -> Net-(IC701-YB2)
- IC701 pad 12: Net-(IC701-1Y3) -> Net-(IC701-YB1)
- IC701 pad 13: Net-(IC701-2A2) -> +3.3V
- IC701 pad 14: Net-(IC701-1Y2) -> GND
- IC701 pad 3: Net-(IC701-2Y0) -> Net-(IC701-A2)
- IC701 pad 4: Net-(IC701-1A1) -> Net-(IC701-A3)
- IC701 pad 5: Net-(IC701-2Y1) -> unconnected-(IC701-YA4-Pad5)
- IC701 pad 6: Net-(IC701-1A2) -> GND
- IC701 pad 7: Net-(IC701-2Y2) -> GND
- IC701 pad 8: Net-(IC701-1A3) -> unconnected-(IC701-B4-Pad8)
- IC701 pad 9: Net-(IC701-2Y3) -> unconnected-(IC701-n.c.-Pad9)
- IC702 pad 1: Net-(IC702-MOD) -> GND
- IC702 pad 2: GND -> Net-(IC702-1A0)
- IC702 pad 3: +3.3V -> Net-(IC702-2Y0)
- IC702 pad 4: GND -> Net-(IC702-1A1)
- IC702 pad 5: +3.3V -> Net-(IC702-2Y1)
- IC702 pad 6: Net-(IC701-2A3) -> Net-(IC702-1A2)
- J701 pad 1: +3.3V -> Net-(IC701-VCC(A))
- J701 pad 3: GND -> Net-(IC701-A2)
- J702 pad 1: Net-(IC701-2Y0) -> +3.3V
- J703 pad 1: Net-(J703-Pin_1) -> Net-(IC702-2Y0)
- J704 pad 2: Net-(IC701-1A2) -> Net-(IC702-1A1)
- J705 pad 1: Net-(IC701-2Y1) -> Net-(IC702-2Y1)
- J706 pad 1: Net-(IC701-2Y2) -> +3.3V
- J707 pad 1: Net-(IC701-2Y3) -> Net-(IC702-2Y2)
- J709 pad 1: +3.3V -> Net-(IC702-2Y3)
- L301 pad 2: Net-(C306-Pad2) -> Net-(C309-Pad2)
- L501 pad 2: /Oscillator Splitter/Oscillator In - -> /Oscillator Splitter/Oscillator In +
- L502 pad 2: /Oscillator Splitter/Oscillator In + -> /Oscillator Splitter/Oscillator In -
- R201 pad 1: Net-(D202-K) -> GND
- R201 pad 2: GND -> /IO Interface/Power Enable
- R202 pad 1: Net-(D203-K) -> Net-(Q201-G)
- R203 pad 1: /power/USB Power -> Net-(D202-K)
- R203 pad 2: /power/Power Faulty -> GND
- R204 pad 1: Net-(D204-K) -> Net-(D203-K)
- R204 pad 2: /power/Power Faulty -> /IO Interface/Power Faulty Out
- R205 pad 1: Net-(U201-PGFB) -> Net-(D204-K)
- R205 pad 2: +3.3V -> GND
- R207 pad 1: GND -> Net-(U201-PGFB)
- R207 pad 2: Net-(U201-ILIM) -> +3.3V
- R208 pad 2: Net-(U201-PGFB) -> Net-(U201-ILIM)
- R209 pad 1: Net-(D205-K) -> GND
- R209 pad 2: GND -> Net-(U201-PGFB)
- R210 pad 1: GND -> Net-(D205-K)
- R210 pad 2: Net-(U201-SET) -> GND
- R211 pad 1: Net-(Q201-G) -> GND
- R211 pad 2: GND -> Net-(U201-SET)
- R301 pad 1: Net-(IC301-VCC1) -> Net-(IC302-VCC1)
- R302 pad 2: Net-(IC301-RFOUT) -> Net-(IC302-RFOUT)
- R303 pad 1: Net-(D301-K) -> GND
- R303 pad 2: GND -> /IO Interface/PA Enable
- R304 pad 1: /IO Interface/PA DET Output -> Net-(D301-K)
- R501 pad 1: /Phase locked loop/PLL: Lock Detect -> /IO Interface/PLL: Power Down
- R501 pad 2: Net-(D501-A) -> +3.3V
- R502 pad 1: /IO Interface/SPI: Load Enable -> /IO Interface/PLL: Power Down
- R503 pad 1: /IO Interface/SPI: DATA -> /IO Interface/PLL: Chip Enable
- R503 pad 2: GND -> +3.3V
- R504 pad 1: /IO Interface/SPI: CLK -> /IO Interface/SPI: Load Enable
- R504 pad 2: GND -> +3.3V
- R505 pad 2: +3.3V -> GND
- R506 pad 1: /IO Interface/PLL: Chip Enable -> /IO Interface/SPI: DATA
- R506 pad 2: +3.3V -> GND
- R507 pad 1: Net-(C514-Pad1) -> /IO Interface/SPI: CLK
- R507 pad 2: Net-(U501-RF_OUT_A+) -> GND
- R508 pad 1: /IO Interface/PLL: Power Down -> /IO Interface/PLL: Lock Detect Out
- R508 pad 2: +3.3V -> Net-(D501-A)
- R509 pad 1: /IO Interface/PLL: Power Down -> Net-(C511-Pad1)
- R509 pad 2: GND -> Net-(U501-RF_OUT_A+)
- R510 pad 1: Net-(C515-Pad1) -> Net-(C512-Pad1)
- R511 pad 2: Net-(C516-Pad1) -> Net-(C513-Pad1)
- R513 pad 2: Net-(C521-Pad1) -> Net-(C517-Pad1)
- R701 pad 1: /IO Interface/Power Enable -> Net-(IC701-YB1)
- R701 pad 2: Net-(IC701-1Y0) -> /IO Interface/SPI: DATA
- R702 pad 1: /IO Interface/PLL: Power Down -> Net-(IC701-YB2)
- R702 pad 2: Net-(IC701-1Y2) -> /IO Interface/SPI: CLK
- R703 pad 1: /IO Interface/PA Enable -> Net-(IC701-YB3)
- R703 pad 2: Net-(IC701-1Y1) -> /IO Interface/SPI: Load Enable
- R704 pad 1: /IO Interface/PLL: Chip Enable -> /IO Interface/Power Enable
- R704 pad 2: Net-(IC701-1Y3) -> Net-(IC702-1Y0)
- R705 pad 1: Net-(IC701-2A2) -> Net-(IC702-2A0)
- R705 pad 2: /IO Interface/PLL: MUXOUT -> /IO Interface/PLL: Lock Detect Out
- R706 pad 1: Net-(IC701-2A0) -> /IO Interface/PA Enable
- R706 pad 2: /IO Interface/PLL: Lock Detect Out -> Net-(IC702-1Y1)
- R707 pad 1: Net-(IC701-2A1) -> Net-(IC702-2A1)
- R708 pad 1: +3.3V -> /IO Interface/PLL: Power Down
- R708 pad 2: GND -> Net-(IC702-1Y2)
- R709 pad 1: Net-(IC702-MOD) -> Net-(IC702-2A2)
- R709 pad 2: /IO Interface/PA DET Output -> /IO Interface/PLL: MUXOUT
- R710 pad 1: Net-(U703-B1) -> /IO Interface/PLL: Chip Enable
- R710 pad 2: /IO Interface/SPI: DATA -> Net-(IC702-1Y3)
- R711 pad 2: /IO Interface/SPI: CLK -> /IO Interface/PA DET Output
- R712 pad 1: Net-(U703-B3) -> +3.3V
- R712 pad 2: /IO Interface/SPI: Load Enable -> GND
- SW201 pad 2: Net-(D203-A) -> Net-(D204-A)
- U501 pad 16: +3.3V -> Net-(C503-Pad1)
- U501 pad 17: +3.3V -> Net-(C503-Pad1)
- U501 pad 25: /Phase locked loop/PLL: Lock Detect -> /IO Interface/PLL: Lock Detect Out
- Y501 pad 4: +3.3V -> Net-(Y501-VDD)
Routing:
- net /power/Power Faulty: track 23.5 -> 0.00 mm, vias 3 -> 0
- net Net-(D203-A): track 19.3 -> 0.00 mm
- net (no net): track 20.5 -> 39.3 mm
- net /power/USB Power: track 64.5 -> 81.1 mm
- net Net-(IC302-RFOUT): track 0.00 -> 6.11 mm
- net Net-(IC302-LO): track 6.11 -> 0.00 mm
- net Net-(IC301-RF): track 0.00 -> 5.51 mm, vias 0 -> 4
- net Net-(IC302-IF): track 4.53 -> 0.00 mm
- net unconnected-(FL402-GROUND_1-Pad1): track 4.21 -> 0.00 mm, vias 2 -> 0
- net Net-(C306-Pad2): track 4.12 -> 0.00 mm
- net Net-(IC302-VCC1): track 0.00 -> 3.95 mm, vias 0 -> 2
- net /IO Interface/PA Enable: track 32.6 -> 36.4 mm, vias 1 -> 3
- net Net-(IC301-LO): track 0.00 -> 3.37 mm, vias 0 -> 2
- net Net-(U201-SET): track 17.3 -> 14.0 mm, vias 2 -> 0
- net Net-(D205-K): track 7.66 -> 4.39 mm, vias 2 -> 0
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Other:
- board size 179.2 x 68.5 mm -> 264.6 x 68.5 mm

Commit message: updated layout
Parts:
- removed IC702: 74LVC244AD-Q100J, My Footprints:SOIC127P1032X265-20N
- added IC704: 74LVC244AD-Q100J, My Footprints:SOIC127P1032X265-20N, F.Cu at (251.1, 93.0)
- added Q701: 2N7002, Package_TO_SOT_SMD:SOT-23, F.Cu at (254.0, 117.8)
- added R713: 10k, Resistor_SMD:R_0603_1608Metric, F.Cu at (263.5, 116.8)
- added R714: 10k, Resistor_SMD:R_0603_1608Metric, F.Cu at (263.5, 112.5)
- added R715: 10k, Resistor_SMD:R_0603_1608Metric, F.Cu at (263.5, 108.2)
- added R716: 10k, Resistor_SMD:R_0603_1608Metric, F.Cu at (263.6, 121.2)
- added R717: 10k, Resistor_SMD:R_0603_1608Metric, F.Cu at (248.8, 120.0)
- moved J703 179.9 mm to (273.8, 95.2), turned to -90 degrees
- moved R202 174.3 mm to (37.0, 123.7), turned to -90 degrees
- moved C205 167.5 mm to (43.4, 76.3)
- moved J709 165.7 mm to (273.8, 71.2), turned to -90 degrees
- moved J707 165.1 mm to (273.8, 79.2), turned to -90 degrees
- moved J706 163.7 mm to (276.3, 83.0), turned to -90 degrees
- moved J708 153.7 mm to (276.3, 75.2), turned to -90 degrees
- moved C703 149.8 mm to (245.1, 82.2), turned to 180 degrees
- moved IC701 146.6 mm to (254.3, 110.8), turned to 180 degrees
- moved J701 143.7 mm to (271.8, 118.6), turned to 180 degrees
- moved R712 141.8 mm to (251.1, 76.2), turned to 180 degrees
- moved J702 139.1 mm to (276.2, 99.0), turned to -90 degrees
- moved R711 131.5 mm to (238.3, 68.7), turned to 180 degrees
- moved J705 130.9 mm to (273.8, 86.7), turned to -90 degrees
- moved J704 130.3 mm to (276.3, 90.7), turned to -90 degrees
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Connections:
- net /power/USB Power renamed /power/Power Raw
- net Net-(C511-Pad1) renamed /Phase locked loop/Ox Blocked +
- net Net-(C512-Pad1) renamed /Phase locked loop/Ox Blocked -
- net Net-(FL301-IN/OUT) renamed /transmitter/RF Out
- net Net-(U501-RF_OUT_A+) renamed /Phase locked loop/Ox +
- net Net-(U501-RF_OUT_A-) renamed /Phase locked loop/Ox -
- IC701 pad 14: GND -> Net-(IC701-~{OE})
- U602 pad 5: /Oscillator Splitter/Oscillator In + -> /Oscillator Splitter/Oscillator In -
- U602 pad 6: /Oscillator Splitter/Oscillator In - -> /Oscillator Splitter/Oscillator In +
Routing:
- net GND: track 280.6 -> 185.7 mm, vias 121 -> 71
- net +3.3V: track 30.4 -> 76.4 mm, vias 13 -> 0
- net +5V: track 165.0 -> 121.7 mm, vias 52 -> 27
- net Net-(IC704-2Y3): track 0.00 -> 31.0 mm
- net Net-(IC701-VCC(A)): track 0.00 -> 27.9 mm
- net Net-(IC704-1A3): track 0.00 -> 27.9 mm
- net Net-(IC703-MOD): track 0.00 -> 27.4 mm
- net Net-(IC704-2Y2): track 0.00 -> 25.0 mm
- net Net-(IC704-1A2): track 0.00 -> 22.7 mm
- net /IO Interface/PLL: Power Down: track 0.00 -> 22.5 mm
- net Net-(IC301-RFOUT): track 22.5 -> 0.00 mm
- net Net-(D204-A): track 0.00 -> 21.4 mm
- net Net-(IC704-2Y1): track 0.00 -> 20.8 mm
- net /power/Power Raw: track 81.1 -> 60.7 mm, vias 2 -> 0
- net Net-(IC704-1Y3): track 0.00 -> 20.3 mm
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- removed copper zone on F.Cu, net +5V
Other:
- board text added: "3.3V Faulty"
- board text added: "Low In/Out High"
- board text added: "PA Detect"
- board text added: "PLL Down"
- board text added: "PLL Enable"
- board text added: "PLL Lock"
- board text added: "SPI: GND Enable Clock Data IO Vcc <=3.3V"
- board text added: "TODO: - via sticthicng with ground plane"
- board text added: "git.ieem-ka.de/Jax/ sdr-analog-frontend"
- board text added: "{ {dblquote}ViaStitching{dblquote}: {dblquote}0.2{dblquote}, {dblquote}stitch_zone_0{dblquote}: { {dblquote}HSpacing{dblquote}: {dblquote}100{dblquote}, {dblquote}VSpacing{dblquote}: {dblquote}100{dblquote}, {dblquote}HOffset{dblquote}: {dblquote}0{dblquote}, {dblquote}VOffset{dblquote}: {dblquote}0{dblquote}, {dblquote}Clearance{dblquote}: {dblquote}0{dblquote}, {dblquote}Randomize{dblquote}: fa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"
- board text removed: "Digital In"
- board text removed: "Digital Out"
- board text removed: "High"
- board text removed: "Low"
- board text removed: "PLL Chip Enable"
- board text removed: "PLL Lock Detect"
- board text removed: "PLL Power Down"
- board text removed: "PLL: Lock Detect"
- board text removed: "SPI: Data Clock Enable"
- board text removed: "TODO: - via fencing - via sticthicng with ground plane - component values on silkscreen"
- board text removed: "https://git.ieem-ka.de/Jax/sdr-analog-frontend"
- board text removed: "{ "ViaStitching": "0.2", "stitch_zone_0": { "HSpacing": "40", "VSpacing": "40", "HOffset": "0", "VOffset": "0", "Clearance": "0", "Randomize": false }, "stitch_zone_1": { "HSpacing": "100", "VSpacing": "100", "HOffset": "0", "VOffset": "0", "Clearance": "0", "Randomize": false } }"

Commit message: updated layout
Parts:
- moved J103 94.6 mm to (139.0, 129.4), turned to -90 degrees
- moved C406 91.2 mm to (130.0, 91.3), turned to 180 degrees
- moved J101 88.5 mm to (155.1, 66.7), turned to 90 degrees
- moved C403 83.2 mm to (139.0, 123.2), turned to 90 degrees
- moved C601 80.3 mm to (88.1, 83.8), turned to 0 degrees
- moved C404 78.9 mm to (138.7, 115.1)
- moved C602 78.7 mm to (88.1, 87.5), turned to 180 degrees
- moved L401 78.3 mm to (142.0, 106.5)
- moved FL401 78.2 mm to (139.0, 118.9)
- moved IC402 77.5 mm to (138.7, 93.8), turned to 0 degrees
- moved IC401 76.7 mm to (140.0, 110.7)
- moved FL402 76.0 mm to (148.5, 82.3), turned to 180 degrees
- moved C401 76.0 mm to (150.6, 98.7), turned to -90 degrees
- moved C402 74.9 mm to (149.0, 106.5)
- moved C405 74.3 mm to (155.2, 76.6)
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Routing:
- net GND: track 185.7 -> 20.3 mm, vias 71 -> 0
- net /IO Interface/Power Enable: track 28.4 -> 179.8 mm, vias 1 -> 4
- net /IO Interface/Power Faulty Out: track 9.28 -> 147.5 mm, vias 0 -> 2
- net /IO Interface/PA DET Output: track 32.1 -> 152.3 mm, vias 1 -> 2
- net /IO Interface/PLL: Power Down: track 22.5 -> 138.5 mm, vias 0 -> 2
- net /IO Interface/PLL: MUXOUT: track 0.00 -> 109.5 mm, vias 0 -> 2
- net /IO Interface/PLL: Lock Detect Out: track 15.5 -> 117.1 mm, vias 0 -> 2
- net /IO Interface/PLL: Chip Enable: track 11.9 -> 111.0 mm, vias 0 -> 2
- net /IO Interface/PA Enable: track 32.6 -> 125.7 mm, vias 1 -> 2
- net /IO Interface/SPI: CLK: track 12.6 -> 87.5 mm, vias 0 -> 2
- net /IO Interface/SPI: Load Enable: track 17.6 -> 90.2 mm, vias 0 -> 2
- net /IO Interface/SPI: DATA: track 9.92 -> 75.7 mm, vias 0 -> 2
- net (no net): track 55.2 -> 0.00 mm
- net +5V: track 121.7 -> 81.6 mm, vias 27 -> 74
- net Net-(FL402-RF_IN): track 36.0 -> 7.17 mm
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- added copper zone on F.Cu, net +3.3V
- added copper zone on F.Cu, net +5V
- added copper zone on F.Cu, net GND
Other:
- board size 264.6 x 68.5 mm -> 204.7 x 68.5 mm
- board text added: "High In/Out Low"
- board text added: "IC601"
- board text added: "On Silkscreen: Assembly Info is placed in left->right or bot->top direction relative to this text. User Info is placed right->left or top->bot relative to this text."
- board text added: "Rx In <- 2.4 - 2.5 GHz"
- board text added: "Rx Out <- 0.9 - 1 GHz"
- board text added: "SPI: IO Vcc <=3.3V Data Clock Enable GND"
- board text added: "TODO: - top layer pour power rails - top layer fix ground to top layer pour - via sticthicng"
- board text added: "Tx In -> 0.9 - 1 GHz"
- board text added: "Tx Out -> 2.4 - 2.5 GHz"
- board text removed: "Low In/Out High"
- board text removed: "Rx: In <-"
- board text removed: "Rx: Out <-"
- board text removed: "SPI: GND Enable Clock Data IO Vcc <=3.3V"
- board text removed: "TODO: - via sticthicng with ground plane"
- board text removed: "Tx: In -> 0.9 - 1 GHz"
- board text removed: "Tx: Out -> 2.4 - 2.5 GHz"
