File: pcb/main_v2/main_v2.kicad_pcb (KiCad board)
At the start: 4 copper layers, 204.7 x 68.5 mm, 182 parts, among them IC201 AP22811AW5-7, IC301 RMS-30+, IC302 SE2576L-R, IC401 HMC374, IC402 RMS-30+, IC601 PSA4-5043+, IC602 PSA4-5043+, IC701 74LVC4T3144PWJ, IC703 LTC6992CS6-4#TRMPBF, IC704 74LVC244AD-Q100J, J101 Conn_Coaxial, J102 Conn_Coaxial, J103 Conn_Coaxial, J104 Conn_Coaxial, J201 Barrel_Jack, J701 Conn_01x05_Pin, J702 Conn_01x03_Pin, J703 Conn_01x01_Pin, J704 Conn_01x03_Pin, J705 Conn_01x01_Pin, J706 Conn_01x03_Pin, J707 Conn_01x01_Pin, J708 Conn_01x03_Pin, J709 Conn_01x01_Pin, Q201 DMP3068L-7, Q701 2N7002, SW201 SW_DIP_x01, U201 LT3042xMSE, U501 ADF4351, U601 PD0922J5050D2HF, U602 XMB0220K1-50100G, Y501 ATX-11-F-26.000MHZ-F05-T

Commit message: finished layout
Parts:
- added C409: 15 pF, Capacitor_SMD:C_0402_1005Metric, F.Cu at (152.7, 73.7)
- added D401: SKY16602-632LF, My Footprints:SKY16602632LF, F.Cu at (158.6, 76.3)
- added J301: CONMHF1-SMD-T, My Footprints:CONMHF1SMDT, F.Cu at (61.7, 90.9)
- added J401: CONMHF1-SMD-T, My Footprints:CONMHF1SMDT, F.Cu at (135.4, 104.5)
- added J601: CONMHF1-SMD-T, My Footprints:CONMHF1SMDT, F.Cu at (86.7, 93.4)
- added J602: CONMHF1-SMD-T, My Footprints:CONMHF1SMDT, F.Cu at (125.2, 82.6)
- added L402: 12 nH, Inductor_SMD:L_0402_1005Metric, F.Cu at (148.8, 73.7)
- added R213: 100k, Resistor_SMD:R_0603_1608Metric, F.Cu at (35.3, 88.3)
- added TP206: TestPoint, TestPoint:TestPoint_Pad_D1.0mm, F.Cu at (45.6, 91.8)
- moved D205 19.1 mm to (26.6, 107.6)
- moved R210 19.1 mm to (26.6, 103.9)
- moved C524 14.8 mm to (102.0, 101.0), turned to 90 degrees
- moved R207 11.5 mm to (38.5, 110.0), turned to 90 degrees
- moved C205 10.6 mm to (51.5, 83.2), turned to -90 degrees
- moved R212 10.1 mm to (37.3, 91.7), turned to 0 degrees
- moved L502 8.26 mm to (103.2, 104.7), turned to -90 degrees
- moved C405 7.13 mm to (159.3, 82.4)
- moved D202 6.44 mm to (42.7, 75.0)
- moved R203 6.44 mm to (38.7, 75.0)
- moved C207 4.80 mm to (40.4, 99.3), turned to -90 degrees
- moved C530 4.80 mm to (93.1, 127.3), turned to -90 degrees
- moved TP205 4.77 mm to (38.7, 112.7), turned to 180 degrees
- moved R303 4.66 mm to (63.4, 99.4)
- moved R208 4.58 mm to (31.6, 97.5)
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Connections:
- C405 pad 2: /receiver/Rx Out -> Net-(D401-RF_IN)
- R301 pad 1: Net-(IC302-VCC1) -> +5V
- R301 pad 2: +5V -> Net-(IC302-VCC1)
Routing:
- net GND: track 20.3 -> 133.2 mm, vias 0 -> 411
- net +5V: track 81.6 -> 53.8 mm, vias 74 -> 341
- net Net-(U201-PGFB): track 7.57 -> 21.2 mm, vias 0 -> 2
- net +3.3V: track 100.5 -> 88.2 mm, vias 49 -> 319
- net /transmitter/Filtered Tx: track 6.95 -> 17.4 mm
- net Net-(D401-PAD): track 0.00 -> 6.93 mm
- net Net-(Y501-VDD): track 16.9 -> 11.9 mm
- net Net-(U201-SET): track 11.2 -> 6.49 mm
- net Net-(D401-RF_IN): track 0.00 -> 4.61 mm
- net /Oscillator Splitter/Oscillator Tx: track 2.94 -> 7.40 mm
- net /receiver/amplified Rx: track 6.57 -> 10.6 mm
- net Net-(U201-ILIM): track 8.21 -> 4.37 mm
- net /Oscillator Splitter/Oscillator In -: track 4.52 -> 8.28 mm
- net /IO Interface/PLL: Lock Detect Out: track 117.1 -> 120.6 mm
- net /Oscillator Splitter/Oscillator Rx: track 7.16 -> 10.2 mm
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Other:
- board text added: "5V Faulty"
- board text added: "Digital I/O"
- board text added: "On Silkscreen: Assembly Info is placed in left->right or bot->top direction relative to this text. User Info is placed right->left or top->bot relative to this text. Example:"
- board text added: "TODO: - via sticthicng top ground"
- board text added: "This is Assembly Info"
- board text added: "This is User Info"
- board text added: "{ "ViaStitching": "0.2", "stitch_zone_0": { "HSpacing": "3", "VSpacing": "3", "HOffset": "0", "VOffset": "0", "Clearance": "0", "Randomize": false } }"
- board text removed: "On Silkscreen: Assembly Info is placed in left->right or bot->top direction relative to this text. User Info is placed right->left or top->bot relative to this text."
- board text removed: "TODO: - top layer pour power rails - top layer fix ground to top layer pour - via sticthicng"
- board text removed: "{ {dblquote}ViaStitching{dblquote}: {dblquote}0.2{dblquote}, {dblquote}stitch_zone_0{dblquote}: { {dblquote}HSpacing{dblquote}: {dblquote}100{dblquote}, {dblquote}VSpacing{dblquote}: {dblquote}100{dblquote}, {dblquote}HOffset{dblquote}: {dblquote}0{dblquote}, {dblquote}VOffset{dblquote}: {dblquote}0{dblquote}, {dblquote}Clearance{dblquote}: {dblquote}0{dblquote}, {dblquote}Randomize{dblquote}: fa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"

Commit message: minor documentaion updates
Parts:
- moved R714 2.12 mm to (203.4, 112.8)
Routing:
- net GND: track 133.2 -> 157.8 mm, vias 411 -> 790
- net +3.3V: track 88.2 -> 90.2 mm, vias 319 -> 124
- net Net-(IC701-A2): track 16.5 -> 15.6 mm
- net +5V: vias 341 -> 159
Other:
- board text removed: "TODO: - via sticthicng top ground"
