File: pcb/main_v2/splitter.kicad_sch (KiCad schematic)
At the start: 15 parts, among them IC601 PSA4-5043+, IC602 PSA4-5043+, U602 XMB0220K1-50100G, U701 PD0922J5050D2HF

Commit message: updated io schematic
Parts:
- renumbered C631 to C601, C630 to C602, C629 to C603, C633 to C604, C634 to C605, C632 to C606, L603 to L601, L605 to L602, R702 to R601, R701 to R602, U701 to U601
Changed lines of the file:
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@@
 		(in_pos_files yes)
 		(dnp no)
-		(property "Reference" "R701"
+		(property "Reference" "R602"
 			(at 224.79 71.12 90)
 			(show_name no)
@@
 			(project "main_v2"
 				(path "/0599865e-4bed-44f1-b46e-4b55335b49b2/b6e6140a-6309-4e0e-b6e0-c9d1e1fed4e9"
-					(reference "R701")
+					(reference "R602")
 					(unit 1)
 				)
@@
 		(dnp no)
 		(fields_autoplaced yes)
-		(property "Reference" "#PWR0643"
+		(property "Reference" "#PWR0606"
 			(at 110.49 118.11 0)
 			(hide yes)
@@
 			(project "main_v2"
 				(path "/0599865e-4bed-44f1-b46e-4b55335b49b2/b6e6140a-6309-4e0e-b6e0-c9d1e1fed4e9"
-					(reference "#PWR0643")
+					(reference "#PWR0606")
 					(unit 1)
 				)
@@
 		(dnp no)
 		(fields_autoplaced yes)
-		(property "Reference" "#PWR0701"
+		(property "Reference" "#PWR0603"
 			(at 251.46 53.34 0)
 			(hide yes)
@@
 			(project "main_v2"
 				(path "/0599865e-4bed-44f1-b46e-4b55335b49b2/b6e6140a-6309-4e0e-b6e0-c9d1e1fed4e9"
-					(reference "#PWR0701")
+					(reference "#PWR0603")
 					(unit 1)
 				)
@@
 		(dnp no)
 		(fields_autoplaced yes)
-		(property "Reference" "U701"
+		(property "Reference" "U601"
 			(at 226.06 43.18 0)
 			(show_name no)
@@
 			(project "main_v2"
 				(path "/0599865e-4bed-44f1-b46e-4b55335b49b2/b6e6140a-6309-4e0e-b6e0-c9d1e1fed4e9"
-					(reference "U701")
+					(reference "U601")
 					(unit 1)
 				)
@@
 		(dnp no)
 		(fields_autoplaced yes)
-		(property "Reference" "#PWR0634"
+		(property "Reference" "#PWR0604"
 			(at 97.79 58.42 0)
 			(hide yes)
@@
 			(project "main_v2"
 				(path "/0599865e-4bed-44f1-b46e-4b55335b49b2/b6e6140a-6309-4e0e-b6e0-c9d1e1fed4e9"
-					(reference "#PWR0634")
+					(reference "#PWR0604")
 					(unit 1)
 				)
@@
 		(dnp no)
 		(fields_autoplaced yes)
-		(property "Reference" "#PWR0642"
+		(property "Reference" "#PWR0609"
 			(at 105.41 133.35 0)
 			(hide yes)
@@
 			(project "main_v2"
 				(path "/0599865e-4bed-44f1-b46e-4b55335b49b2/b6e6140a-6309-4e0e-b6e0-c9d1e1fed4e9"
-					(reference "#PWR0642")
+					(reference "#PWR0609")
 					(unit 1)
 				)
@@
 		(in_pos_files yes)
 		(dnp no)
-		(property "Reference" "R702"
+		(property "Reference" "R601"
 			(at 232.156 39.116 90)
 			(show_name no)
@@
 			(project "main_v2"
 				(path "/0599865e-4bed-44f1-b46e-4b55335b49b2/b6e6140a-6309-4e0e-b6e0-c9d1e1fed4e9"
-					(reference "R702")
+					(reference "R601")
 					(unit 1)
 				)
@@
 		(dnp no)
 		(fields_autoplaced yes)
-		(property "Reference" "#PWR0644"
+		(property "Reference" "#PWR0612"
 			(at 50.8 176.53 0)
 			(hide yes)
@@
 			(project "main_v2"
 				(path "/0599865e-4bed-44f1-b46e-4b55335b49b2/b6e6140a-6309-4e0e-b6e0-c9d1e1fed4e9"
-					(reference "#PWR0644")
+					(reference "#PWR0612")
 					(unit 1)
 				)
@@
 		(in_pos_files yes)
 		(dnp no)
-		(property "Reference" "L603"
+		(property "Reference" "L601"
 			(at 100.33 125.7299 0)
 			(show_name no)
@@
 			(project "main_v2"
 				(path "/0599865e-4bed-44f1-b46e-4b55335b49b2/b6e6140a-6309-4e0e-b6e0-c9d1e1fed4e9"
-					(reference "L603")
+					(reference "L601")
 					(unit 1)
 				)
@@
 		(in_pos_files yes)
 		(dnp no)
-		(property "Reference" "C630"
+		(property "Reference" "C602"
 			(at 123.19 137.16 0)
 			(show_name no)
@@
 			(project "main_v2"
 				(path "/0599865e-4bed-44f1-b46e-4b55335b49b2/b6e6140a-6309-4e0e-b6e0-c9d1e1fed4e9"
-					(reference "C630")
+					(reference "C602")
 					(unit 1)
 				)
@@
 		(dnp no)
 		(fields_autoplaced yes)
-		(property "Reference" "#PWR0648"
+		(property "Reference" "#PWR0607"
 			(at 110.49 128.27 0)
 			(hide yes)
@@
 			(project "main_v2"
 				(path "/0599865e-4bed-44f1-b46e-4b55335b49b2/b6e6140a-6309-4e0e-b6e0-c9d1e1fed4e9"
-					(reference "#PWR0648")
+					(reference "#PWR0607")
 					(unit 1)
 				)
@@
 		(dnp no)
 		(fields_autoplaced yes)
-		(property "Reference" "#PWR0647"
+		(property "Reference" "#PWR0611"
 			(at 111.76 173.99 0)
 			(hide yes)
@@
 			(project "main_v2"
 				(path "/0599865e-4bed-44f1-b46e-4b55335b49b2/b6e6140a-6309-4e0e-b6e0-c9d1e1fed4e9"
-					(reference "#PWR0647")
+					(reference "#PWR0611")
 					(unit 1)
 				)
@@
 		(in_pos_files yes)
 		(dnp no)
-		(property "Reference" "C633"
+		(property "Reference" "C604"
 			(at 118.11 162.56 0)
 			(show_name no)
@@
 			(project "main_v2"
 				(path "/0599865e-4bed-44f1-b46e-4b55335b49b2/b6e6140a-6309-4e0e-b6e0-c9d1e1fed4e9"
-					(reference "C633")
+					(reference "C604")
 					(unit 1)
 				)
@@
 		(dnp no)
 		(fields_autoplaced yes)
-		(property "Reference" "#PWR0645"
+		(property "Reference" "#PWR0613"
 			(at 106.68 179.07 0)
 			(hide yes)
@@
 			(project "main_v2"
 				(path "/0599865e-4bed-44f1-b46e-4b55335b49b2/b6e6140a-6309-4e0e-b6e0-c9d1e1fed4e9"
-					(reference "#PWR0645")
+					(reference "#PWR0613")
 					(unit 1)
 				)
@@
 		(in_pos_files yes)
 		(dnp no)
-		(property "Reference" "C629"
+		(property "Reference" "C603"
 			(at 44.45 139.7 0)
 			(show_name no)
@@
 			(project "main_v2"
 				(path "/0599865e-4bed-44f1-b46e-4b55335b49b2/b6e6140a-6309-4e0e-b6e0-c9d1e1fed4e9"
-					(reference "C629")
+					(reference "C603")
 					(unit 1)
 				)
@@
 		(in_pos_files yes)
 		(dnp no)
-		(property "Reference" "C631"
+		(property "Reference" "C601"
 			(at 116.84 116.84 0)
 			(show_name no)
@@
 			(project "main_v2"
 				(path "/0599865e-4bed-44f1-b46e-4b55335b49b2/b6e6140a-6309-4e0e-b6e0-c9d1e1fed4e9"
-					(reference "C631")
+					(reference "C601")
 					(unit 1)
 				)
@@
 		(dnp no)
 		(fields_autoplaced yes)
-		(property "Reference" "#PWR0646"
+		(property "Reference" "#PWR0610"
 			(at 111.76 163.83 0)
 			(hide yes)
@@
 			(project "main_v2"
 				(path "/0599865e-4bed-44f1-b46e-4b55335b49b2/b6e6140a-6309-4e0e-b6e0-c9d1e1fed4e9"
-					(reference "#PWR0646")
+					(reference "#PWR0610")
 					(unit 1)
 				)
@@
 		(dnp no)
 		(fields_autoplaced yes)
-		(property "Reference" "#PWR0641"
+		(property "Reference" "#PWR0608"
 			(at 49.53 130.81 0)
 			(hide yes)
@@
 			(project "main_v2"
 				(path "/0599865e-4bed-44f1-b46e-4b55335b49b2/b6e6140a-6309-4e0e-b6e0-c9d1e1fed4e9"
-					(reference "#PWR0641")
+					(reference "#PWR0608")
 					(unit 1)
 				)
@@
 		(dnp no)
 		(fields_autoplaced yes)
-		(property "Reference" "#PWR0608"
+		(property "Reference" "#PWR0605"
 			(at 135.89 77.47 0)
 			(hide yes)
@@
 			(project "main_v2"
 				(path "/0599865e-4bed-44f1-b46e-4b55335b49b2/b6e6140a-6309-4e0e-b6e0-c9d1e1fed4e9"
-					(reference "#PWR0608")
+					(reference "#PWR0605")
 					(unit 1)
 				)
@@
 		(dnp no)
 		(fields_autoplaced yes)
-		(property "Reference" "#PWR0640"
+		(property "Reference" "#PWR0601"
 			(at 135.89 29.21 0)
 			(hide yes)
@@
 			(project "main_v2"
 				(path "/0599865e-4bed-44f1-b46e-4b55335b49b2/b6e6140a-6309-4e0e-b6e0-c9d1e1fed4e9"
-					(reference "#PWR0640")
+					(reference "#PWR0601")
 					(unit 1)
 				)
@@
 		(in_pos_files yes)
 		(dnp no)
-		(property "Reference" "L605"
+		(property "Reference" "L602"
 			(at 101.6 171.4499 0)
 			(show_name no)
@@
 			(project "main_v2"
 				(path "/0599865e-4bed-44f1-b46e-4b55335b49b2/b6e6140a-6309-4e0e-b6e0-c9d1e1fed4e9"
-					(reference "L605")
+					(reference "L602")
 					(unit 1)
 				)
@@
 		(in_pos_files yes)
 		(dnp no)
-		(property "Reference" "C634"
+		(property "Reference" "C605"
 			(at 124.46 182.88 0)
 			(show_name no)
@@
 			(project "main_v2"
 				(path "/0599865e-4bed-44f1-b46e-4b55335b49b2/b6e6140a-6309-4e0e-b6e0-c9d1e1fed4e9"
-					(reference "C634")
+					(reference "C605")
 					(unit 1)
 				)
@@
 		(in_pos_files yes)
 		(dnp no)
-		(property "Reference" "C632"
+		(property "Reference" "C606"
 			(at 45.72 185.42 0)
 			(show_name no)
@@
 			(project "main_v2"
 				(path "/0599865e-4bed-44f1-b46e-4b55335b49b2/b6e6140a-6309-4e0e-b6e0-c9d1e1fed4e9"
-					(reference "C632")
+					(reference "C606")
 					(unit 1)
 				)
@@
 		(dnp no)
 		(fields_autoplaced yes)
-		(property "Reference" "#PWR0633"
+		(property "Reference" "#PWR0602"
 			(at 44.45 53.34 0)
 			(hide yes)
@@
 			(project "main_v2"
 				(path "/0599865e-4bed-44f1-b46e-4b55335b49b2/b6e6140a-6309-4e0e-b6e0-c9d1e1fed4e9"
-					(reference "#PWR0633")
+					(reference "#PWR0602")
 					(unit 1)
 				)

Commit message: updated layout
Connections:
- net Oscillator In +: now also U602.6; no longer U602.5
- net Oscillator In -: now also U602.5; no longer U602.6

Commit message: finished layout
Parts:
- added J601, J602: CONMHF1-SMD-T, My Footprints:CONMHF1SMDT, symbol My Symbols:CONMHF1-SMD-T
Connections:
- net GND: now also J601.2 (GND_1), J601.3 (GND_2), J601.4 (GND_3), J602.2 (GND_1), J602.3 (GND_2), J602.4 (GND_3)
- net Oscillator Rx: now also J602.1 (SIGNAL)
- net Oscillator Tx: now also J601.1 (SIGNAL)
Other:
- moved on the sheet: C601, C602, C603, C604, C605, C606, IC601, IC602, L601, L602
