File: pcb/main_v2/main_v2.kicad_sch (KiCad schematic)
At the start: 8 parts, among them J101 Conn_Coaxial, J102 Conn_Coaxial, J103 Conn_Coaxial, J104 Conn_Coaxial

Commit message: added second LNA
Other:
- note added: "More Information about the PCb can be found at: https://git.ieem-ka.de/Jax/sdr-analog-frontend - design documentation - python simulation - KiCad Project with schematic, layout, bom - relevant component library - current issues - ..."
- note added: "TODO: add final BOM, pricelist, order link mit der HKA ilias vorlage"
- note added: "TODO: add thermal vias"
Changed lines of the file:
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@@
 	(generator_version "10.0")
 	(paper "A4")
+	(text "TODO: add final BOM, pricelist, order link\n\nmit der HKA ilias vorlage"
+		(exclude_from_sim no)
+		(at 92.202 117.094 0)
+		(effects
+			(font
+				(size 1.27 1.27)
+			)
+		)
+	)
+	(text "TODO: add thermal vias"
+		(exclude_from_sim no)
+		(at 92.456 108.712 0)
+		(effects
+			(font
+				(size 1.27 1.27)
+			)
+		)
+	)
+	(text "More Information about the PCb can be found at:\nhttps://git.ieem-ka.de/Jax/sdr-analog-frontend\n- design documentation\n- python simulation\n- KiCad Project with schematic, layout, bom\n- relevant component library\n- current issues\n- ..."
+		(exclude_from_sim no)
+		(at 17.78 185.166 0)
+		(effects
+			(font
+				(size 1.27 1.27)
+			)
+			(justify left)
+		)
+	)
 	(text "RFSOC:\nhttps://www.realdigital.org/downloads/15456c97a4fe5a1ee66208c5aa3894bb.pdf\n\nADC:\nmax input power: 14.6 dBm\nattenuation range: 27 dB\ninput bandwith: 6 GHz\n\nDAC:\nMax output power: -18.5 to 6.5 dBm\ncurrent max: 40.5 mA\n"
 		(exclude_from_sim no)

Commit message: added second LNA
Changed lines of the file:
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@@
 	(text "TODO: add final BOM, pricelist, order link\n\nmit der HKA ilias vorlage"
 		(exclude_from_sim no)
-		(at 92.202 117.094 0)
+		(at 91.44 98.044 0)
 		(effects
 			(font
@@
 		)
 	)
-	(text "TODO: add thermal vias"
+	(text "TODO: add thermal vias\n"
 		(exclude_from_sim no)
-		(at 92.456 108.712 0)
+		(at 86.106 118.872 0)
 		(effects
 			(font
