File: pcb/main_v2/pll.kicad_sch (KiCad schematic)
At the start: 53 parts, among them U501 ADF4351, Y501 ATX-11-F-26.000MHZ-F05-T

Commit message: updated project after assembly
Parts:
- C527: value 1nF -> 1 nF
Changed lines of the file:
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@@
 			)
 		)
-		(property "Value" "1nF"
+		(property "Value" "1 nF"
 			(at 127.254 173.228 0)
 			(show_name no)
