File: pcb/main_v2/transmitter.kicad_sch (KiCad schematic)
At the start: 23 parts, among them IC301 RMS-30+, IC302 SE2576L-R

Commit message: finished layout
Parts:
- added J301: CONMHF1-SMD-T, My Footprints:CONMHF1SMDT, symbol My Symbols:CONMHF1-SMD-T
Connections:
- net Filtered Tx: now also J301.1 (SIGNAL)
- net GND: now also J301.2 (GND_1), J301.3 (GND_2), J301.4 (GND_3)

Commit message: added second LNA
Other:
- note added: "Place Thermal Vias for Heat Dissapation!"
Changed lines of the file:
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@@
 	(generator_version "10.0")
 	(paper "A4")
+	(text "Place Thermal Vias for Heat Dissapation!"
+		(exclude_from_sim no)
+		(at 140.208 141.732 0)
+		(effects
+			(font
+				(size 1.27 1.27)
+			)
+		)
+	)
 	(text "Eval Board\nhttps://www.eevblog.com/forum/rf-microwave/2-4ghz-amplifier-quadrature-hybrid-coupler-balanced/?action=dlattach;attach=686451"
 		(exclude_from_sim no)
@@
 					(unit 1)
 				)
+			)
+		)
+	)
+	(symbol
+		(lib_id "Graphic:SYM_Hot_Small")
+		(at 139.7 146.05 0)
+		(unit 1)
+		(body_style 1)
+		(exclude_from_sim yes)
+		(in_bom no)
+		(on_board no)
+		(in_pos_files yes)
+		(dnp no)
+		(fields_autoplaced yes)
+		(property "Reference" "#SYM301"
+			(at 139.7 142.494 0)
+			(hide yes)
+			(show_name no)
+			(do_not_autoplace no)
+			(effects
+				(font
+					(size 1.27 1.27)
+				)
+			)
+		)
+		(property "Value" "SYM_Hot_Small"
+			(at 139.7 149.225 0)
+			(hide yes)
+			(show_name no)
+			(do_not_autoplace no)
+			(effects
+				(font
+					(size 1.27 1.27)
+				)
+			)
+		)
+		(property "Footprint" ""
+			(at 139.7 150.495 0)
+			(hide yes)
+			(show_name no)
+			(do_not_autoplace no)
+			(effects
+				(font
+					(size 1.27 1.27)
+				)
+			)
+		)
+		(property "Datasheet" ""
+			(at 140.462 151.13 0)
+			(hide yes)
+			(show_name no)
+			(do_not_autoplace no)
+			(effects
+				(font
+					(size 1.27 1.27)
+				)
+			)
+		)
+		(property "Description" "Hot surface warning symbol, small"
+			(at 139.7 146.05 0)
+			(hide yes)
+			(show_name no)
+			(do_not_autoplace no)
+			(effects
+				(font
+					(size 1.27 1.27)
+				)
+			)
+		)
+		(instances
+			(project "main_v2"
+				(path "/0599865e-4bed-44f1-b46e-4b55335b49b2/fc4ed8a1-ee18-4353-b821-8d1b4dc84288"
+					(reference "#SYM301")
+					(unit 1)
+				)

Commit message: updated project after assembly
Parts:
- C311: value 3.3 pF -> 3.2 pF
Changed lines of the file:
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@@
 			)
 		)
-		(property "Value" "3.3 pF"
+		(property "Value" "3.2 pF"
 			(at 127 120.65 0)
 			(show_name no)
